File: KicadFiles/PiezzCircuit/PiezzCircuit.sch (KiCad schematic (older format))
At the start: 16 parts, among them J1 PiezoElectricConn, J2 Conn_01x03_Male, J3 ADCInput, J6 Support, J7 ExtSupply, U1 MCP6022, U2 LM385BZ-1.2

Commit message: New project CCS
Parts:
- added C1, C2: 1n, Capacitor_THT:C_Rect_L4.0mm_W2.5mm_P2.50mm, symbol Device:C
- added C3: 1nF, Capacitor_THT:CP_Radial_D5.0mm_P2.00mm, symbol Device:CP
- added C4: 10uF, Capacitor_THT:C_Rect_L4.0mm_W2.5mm_P2.50mm, symbol Device:C
- added R1, R2: 100M, Resistor_THT:R_Axial_DIN0207_L6.3mm_D2.5mm_P10.16mm_Horizontal, symbol Device:R
- added R3, R4: R, Resistor_THT:R_Axial_DIN0207_L6.3mm_D2.5mm_P10.16mm_Horizontal, symbol Device:R
- added U1: MCP6022, MCP602-I_P:DIP787W46P254L927H533Q8, symbol Amplifier_Operational:MCP6022
- added Y1: PiezoElectric, XDCR_SMD10T3R111, symbol SMD10T3R111:SMD10T3R111
Connections:
- net GND: now also C3.2, C4.2, R4.2, U1.4 (V-)
- net VDD: now also C3.1, C4.1, R3.1, U1.8 (V+)
- new net: C1.1, R1.1, U1.1
- new net: C1.2, R1.2, U1.2 (-), Y1.+
- new net: C2.1, R2.1, U1.3 (+), Y1.-
- new net: C2.2, R2.2, U1.6 (-), U1.7
- new net: R3.2, R4.1, U1.5 (+)
