File: KicadFiles/AccCircV2/AccCircV2.sch (KiCad schematic (older format))
At the start: 13 parts, among them J1 AccelConnector, J2 ADCInput, J3 IO, J4 ExtSupply, U1 MCP602, U2 LM385Z-ADJ

Commit message: New project CCS
Parts:
- removed J4: ExtSupply, Connector_PinHeader_2.54mm:PinHeader_1x03_P2.54mm_Horizontal, symbol Connector:Conn_01x03_Male
- removed R3: R, Resistor_THT:R_Axial_DIN0207_L6.3mm_D2.5mm_P10.16mm_Horizontal, symbol Device:R
- added C3: 10uF, Capacitor_THT:CP_Radial_D5.0mm_P2.50mm, symbol Device:CP1
- added D1: 1N4001, Diode_THT:D_DO-41_SOD81_P10.16mm_Horizontal, symbol Diode:1N4001
- added J4: ExternalSupply3V3, Connector_PinHeader_2.54mm:PinHeader_1x02_P2.54mm_Vertical, symbol Connector:Conn_01x02_Male
- added J5: VoltageRefSel, Connector_PinHeader_2.54mm:PinHeader_1x03_P2.54mm_Vertical, symbol Connector:Conn_01x03_Male
- added J6: Solenoid Connector, Connector_PinHeader_2.54mm:PinHeader_1x02_P2.54mm_Vertical, symbol Connector:Conn_01x02_Male
- added J7: ExternalSupply5V, Connector_PinHeader_2.54mm:PinHeader_1x02_P2.54mm_Vertical, symbol Connector:Conn_01x02_Male
- added J8: ControlSig, Connector_PinHeader_2.54mm:PinHeader_1x03_P2.54mm_Vertical, symbol Connector:Conn_01x03_Male
- added Q1: TN0207, Package_TO_SOT_THT:TO-92_Inline, symbol Transistor_FET:2N7000
- added R5: R, Resistor_THT:R_Axial_DIN0207_L6.3mm_D2.5mm_P10.16mm_Horizontal, symbol Device:R
- added R6: 10k, Resistor_THT:R_Axial_DIN0207_L6.3mm_D2.5mm_P10.16mm_Horizontal, symbol Device:R
- added unit 2 of U1
- J1: footprint Connector_PinHeader_2.54mm:PinHeader_1x03_P2.54mm_Horizontal -> Connector_PinHeader_2.54mm:PinHeader_1x03_P2.54mm_Vertical
- renumbered R5 to R3
Connections:
- net labels added: +3.3V, +5V, AccSignal, VolDivider
- net labels removed: VDD
- wire segments 44 -> 70
Other:
- note added: "Control Signals"
- note added: "External Supply 3.3V\n"
- note added: "External Supply 5V\n"
- note added: "OpAmp Supply\n"
- note added: "Solenoid Driver"
- note added: "VoltageRef_HalfSupply"
- note removed: "External Supply\n"
- note removed: "Power Supply\n"
- moved on the sheet: J1, J3

Commit message: some changes
Parts:
- Q1: footprint Package_TO_SOT_THT:TO-92_Inline -> Package_TO_SOT_THT:TO-92L_Inline_Wide
Changed lines of the file:
@@
 F 0 "Q1" H 8905 3596 50  0000 L CNN
 F 1 "TN0207" H 8905 3505 50  0000 L CNN
-F 2 "Package_TO_SOT_THT:TO-92_Inline" H 8900 3475 50  0001 L CIN
+F 2 "Package_TO_SOT_THT:TO-92L_Inline_Wide" H 8900 3475 50  0001 L CIN
 F 3 "https://www.onsemi.com/pub/Collateral/NDS7002A-D.PDF" H 8700 3550 50  0001 L CNN
 	1    8700 3550
